Commit message: eazydrone

File: genesis/drone.urdf (robot description, URDF)
Before this commit: robot cf2_p_variant, 6 links, 6 joints
Joints:
- joint lidar_joint: axis (none) -> 0 0 0

Commit message: lidar

File: genesis/drone.urdf (robot description, URDF)
Before this commit: robot cf2_p_variant, 6 links, 6 joints
Joints:
- joint lidar_joint: origin xyz=0 0 0.03 rpy=0 0 0 -> xyz=0 0 0.2 rpy=0 0 0
